File: hardware/wiflier.sch (KiCad schematic (older format))
At the start: 58 parts, among them CN1 10p, J1 AVRISP6, P1 WS2812, P10 SCL, P11 3V, P12 GND, P13 LED, P14 LED, P15 LED, P16 BAT, P17 TOUT, P2 M0, P21 B+, P24 B-, P3 M1, P32 ESP_UART, P4 M2, P5 M3, P6 ANT, P9 SDA, Q1 7A_20V, Q2 7A_20V, Q3 7A_20V, Q4 7A_20V, U1 MCP1824/3.3, U2 MCP1824/3.3, U3 BMP085, U4 LSM9DS1, U5 ESP8266EX, U6 W25Q80DV, U7 ATTINY441-QFN, X1 26MHz

Commit message: total rework over a lot of stuff, now we have sort of closed loop control.
Parts:
- R3: Cost .011 -> (none); Digikey 1276-4584-1-ND -> (none)
Changed lines of the file:
@@
 LIBS:attiny441
 LIBS:lsm9ds1
-LIBS:wiflier-cache
 EELAYER 27 0
 EELAYER END
@@
 F 2 "NP" V 9330 1900 30  0000 C CNN
 F 3 "~" H 9400 1900 30  0000 C CNN
-F 4 "1276-4584-1-ND" V 9400 1900 60  0001 C CNN "Digikey"
-F 5 ".011" V 9400 1900 60  0001 C CNN "Cost"
+F 4 "~" V 9400 1900 60  0001 C CNN "Digikey"
+F 5 "~" V 9400 1900 60  0001 C CNN "Cost"
 	1    9400 1900
 	0    -1   -1   0
