File: hardware/wiflierB.kicad_pcb (KiCad board)
At the start: 2 copper layers, 37.8 x 21.5 mm, 61 parts, among them CN1 10p, J1 AVRISP6, P1 WS2812, P10 SCL, P11 3V, P12 GND, P13 LED, P14 LED, P15 GND, P16 FLTBAT, P17 TOUT, P18 AVRA0, P2 M0, P21 B+, P24 B-, P3 M1, P32 ESP_UART, P4 M2, P5 M3, P6 ANT, P9 SDA, Q1 7A_20V, Q2 7A_20V, Q3 7A_20V, Q4 7A_20V, U1 MCP1824/3.3, U2 MCP1824/3.3, U3 BMP280, U4 LSM9DS1, U5 ESP8266EX, U6 W25Q80DV, U7 ATTINY441-QFN, X1 26MHz

Commit message: Woah, too many commits to count.  I guess I just havne't committed anything here in a looong time.
Other:
- board text added: "WARNING: UNTESTED DOES NOT MATCH FIRMWARE After testing, inexplicably fails."
- board text removed: "WARNING: UNTESTED DOES NOT MATCH FIRMWARE"
Changed lines of the file:
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@@
     )
   )
-  (gr_text "WARNING: UNTESTED\nDOES NOT MATCH\nFIRMWARE" (at 68.5546 76.708) (layer Cmts.User)
+  (gr_text "WARNING: UNTESTED\nDOES NOT MATCH\nFIRMWARE\nAfter testing, inexplicably fails." (at 68.5546 76.708) (layer Cmts.User)
     (effects (font (size 5.08 5.08) (thickness 0.3)))
   )
