File: hardware/wiflier_EXP_B.kicad_pcb (KiCad board)
At the start: 2 copper layers, 37.8 x 21.5 mm, 61 parts, among them CN1 10p, P1 GPIO2, P10 SCL, P11 3V, P12 GND, P13 LED, P14 LED, P15 LED, P16 BAT, P17 TOUT, P18 PA0, P19 ANT, P2 M0, P21 B+, P24 B-, P3 M1, P32 ESP_UART, P4 M2, P5 M3, P6 ANT, P9 SDA, Q1 7A_20V, Q2 7A_20V, Q3 7A_20V, Q4 7A_20V, U1 MCP1824/3.3, U2 MCP1824/3.0, U3 BMP280, U4 LSM9DS1, U5 ESP8266EX, U6 W25Q16DV, U7 ATTINY841-QFN, X1 26MHz

Commit message: General updates with MPFS thing
Other:
- board text added: "(1) Use lead-based solder paste. Bismuth OK, but ONLY if specifically directed. Some applications cannot use bismuth solder paste. If you use bismuth, mark board indicating as such. (2) Use 1.0mm to 1.2mm thick boards. Do not exceed 1.2mm thickness. (Unless prototyping) (3) ENIG finish recommended. (4) Factory DO NOT populate parts on bottom of board. (5) L1, L2 DO NOT populate. (6) If a wider ch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"
- board text added: "(C) 2014, 2015 C. Lohr WiflierEXP (Rev B)"
- board text added: "1 Inch"
- board text added: "WiflierEXP (Rev B)"
- board text removed: "(C) 2014, 2015 C. Lohr WiflierEXP (Rev A)"
- board text removed: "EXPERIMENTAL DO NOT USE"
- board text removed: "WiflierEXP (Rev A)"
Changed lines of the file:
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@@
     (links 156)
     (no_connects 0)
-    (area 29.172414 49.125999 113.600986 81.278)
+    (area 13.12418 13.081 126.399728 71.257716)
     (thickness 1.6)
-    (drawings 43)
+    (drawings 45)
     (tracks 834)
     (zones 0)
@@
     (nets 42)
   )
-  (page User 139.7 139.7)
+  (page User 139.7 106.68)
   (title_block
     (title Wiflier)
-    (rev -)
+    (rev B)
+    (company "Copyright 2015 <>< Charles Lohr")
   )
   (layers
-    (15 F.Cu signal hide)
+    (15 F.Cu signal)
     (0 B.Cu signal)
     (16 B.Adhes user)
@@
     (pad_to_mask_clearance 0.06858)
     (aux_axis_origin 0 0)
-    (visible_elements FFFFFFEF)
+    (visible_elements FFFFFFFF)
     (pcbplotparams
-      (layerselection 284721153)
+      (layerselection 318275585)
       (usegerberextensions true)
       (excludeedgelayer false)
@@
       (drillshape 0)
       (scaleselection 1)
-      (outputdirectory wiflierEXPA))
+      (outputdirectory wiflierEXPB))
   )
   (net 0 "")
@@
       (effects (font (size 0.762 0.762) (thickness 0.1524)))
     )
-    (fp_text value BMP280 (at 0.2 2.2 90) (layer F.SilkS)
+    (fp_text value BMP280 (at 0.10414 2.12598 90) (layer F.SilkS)
       (effects (font (size 0.762 0.762) (thickness 0.1524)))
     )
@@
     )
   )
-  (gr_text "EXPERIMENTAL DO NOT USE" (at 71.3867 77.978) (layer Cmts.User)
-    (effects (font (size 4 4) (thickness 1)))
-  )
-  (gr_text "WiflierEXP (Rev A)" (at 61.5315 50.1015) (layer F.SilkS)
+  (gr_text "(1) Use lead-based solder paste. Bismuth OK, but ONLY if specifically directed.\n   Some applications cannot use bismuth solder paste.  If you use bismuth, mark\n   board indicating as such.\n(2) Use 1.0mm to 1.2mm thick boards.  Do not exceed 1.2mm thickness.\n   (Unless prototyping)\n(3) ENIG finish recommended.\n(4) Factory DO NOT populate parts on bottom of board.\n(5) L1, L2 DO NOT populate.\n(6) If a wider chip is used for U6, bend leads under." (at 13.28928 14.9987) (layer Cmts.User)
+    (effects (font (size 2.032 1.778) (thickness 0.3302)) (justify left))
+  )
+  (gr_text "1 Inch" (at 61.59246 46.2661) (layer Cmts.User)
+    (effects (font (size 1.5 1.5) (thickness 0.3)))
+  )
+  (gr_line (start 48.895 44.45) (end 74.295 44.45) (angle 90) (layer Cmts.User) (width 0.2))
+  (gr_text "WiflierEXP (Rev B)" (at 61.5315 50.1015) (layer F.SilkS)
     (effects (font (size 0.8128 0.8128) (thickness 0.1651)))
   )
@@
   (gr_line (start 55.05704 54.00294) (end 55.56504 53.49494) (angle 90) (layer B.SilkS) (width 0.2))
   (gr_line (start 55.05704 54.51094) (end 55.05704 54.00294) (angle 90) (layer B.SilkS) (width 0.2))
-  (gr_text "(C) 2014, 2015 C. Lohr\nWiflierEXP (Rev A)" (at 64.5414 54.2036) (layer B.SilkS)
+  (gr_text "(C) 2014, 2015 C. Lohr\nWiflierEXP (Rev B)" (at 64.5414 54.2036) (layer B.SilkS)
     (effects (font (size 0.762 0.762) (thickness 0.1524)) (justify mirror))
   )
