File: hardware/wiflier_EXP_B.sch (KiCad schematic (older format))
At the start: 63 parts, among them CN1 10p, P1 GPIO2, P10 SCL, P11 3V, P12 GND, P13 LED, P14 LED, P15 LED, P16 BAT, P17 TOUT, P18 PA0, P19 ANT, P2 M0, P21 B+, P24 B-, P3 M1, P32 ESP_UART, P4 M2, P5 M3, P6 ANT, P9 SDA, Q1 7A_20V, Q2 7A_20V, Q3 7A_20V, Q4 7A_20V, U1 MCP1824/3.3, U2 MCP1824/3.0, U3 BMP280, U4 LSM9DS1, U5 ESP8266EX, U6 W25Q16DV, U7 ATTINY841-QFN, X1 26MHz

Commit message: General updates with MPFS thing
Parts:
- FB1: value - -> FB_500ma; Cost (none) -> .10; Digikey (none) -> 553-2382-1-ND
Other:
- note added: "Note: Original Design Name was\nQuadcopter_dc4l, Transition Rev D. \nThis is "EXPB" Do not use old\nfirmware on this board."
- note removed: "EXPERIMENTAL\nNO PRODUCTION"
- note removed: "Note: Original Design Name was Quadcopter_dc4l, Transition Rev D"
- moved on the sheet: D1, D2, D3, D4, P2, P3, P4, P5, Q1, Q2, Q3, Q4
