File: wiflier8285/wiflier8285.sch (KiCad schematic (older format))
At the start: 46 parts, among them CN1 1u, CN2 1u, M0 M, M1 M, M2 M, M3 M, P1 USBMicroB-10118194-0001LF, P2 CONN_01X02, P3 I2C, P4 TXRX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

Commit message: Update!
Parts:
- added D7, D8: BLU, SM0805, symbol LED
- added E1, E2: 10u, SM0603, symbol C
- added E3: 100u, C_1206, symbol C
- added R6, R7: 1.5k, SM0603, symbol R
- A1: footprint ANT1206 -> RFANT8010080A3T
- P1: value USBMicroB-10118194-0001LF -> USB
- P2: value CONN_01X02 -> BATTERY
Connections:
- net +3V3: now also E1.2, E2.2
- net BATT: now also E3.2
- net G2: now also D7.2 (A), D8.2 (A)
- net GND: now also E1.1, E2.1, E3.1, R6.1, R7.1
- new net: D7.1 (K), R7.2
- new net: D8.1 (K), R6.2
Other:
- note added: "EXPERIMENTAL\nDO NOT USE\n\nTODO: Add 10u caps + an extra .1u\nTODO: Off-board LEDs"
- note removed: "EXPERIMENTAL\nDO NOT USE\n\nTODO: Add 10u caps + an extra .1u"
Changed lines of the file:
@@
 	1    0    0    -1
 $EndComp
-Wire Wire Line
-	5750 1000 5750 950
-Wire Wire Line
-	5750 950  5600 950
-Wire Wire Line
-	4850 1000 4850 950
-Wire Wire Line
-	4850 950  5000 950
-Wire Wire Line
-	4850 1300 5750 1300
-Wire Wire Line
-	5250 1300 5250 1250
-Connection ~ 5250 1300
-Wire Wire Line
-	5350 1300 5350 1250
-Connection ~ 5350 1300
-Wire Wire Line
-	5600 1300 5600 1350
-Connection ~ 5600 1300
-Wire Wire Line
-	2650 1250 2650 1350
 Text GLabel 1750 2500 0    60   Input ~ 0
 GPIO16
@@
 P 7250 2450
 F 0 "P1" H 7400 2650 60  0000 C CNN
-F 1 "USBMicroB-10118194-0001LF" H 7250 2750 60  0000 C CNN
+F 1 "USB" H 7250 2750 60  0000 C CNN
 F 2 "USBMicroB-10118194-0001LF" H 7250 2500 60  0001 C CNN
 F 3 "" H 7250 2500 60  0001 C CNN
@@
 F 0 "A1" V 1380 1900 50  0000 C CNN
 F 1 "ANTENNA" V 1300 1900 50  0000 C CNN
-F 2 "ANT1206" V 1230 1900 30  0000 C CNN
+F 2 "RFANT8010080A3T" V 1230 1900 30  0000 C CNN
 F 3 "" H 1300 1900 30  0000 C CNN
 	1    1300 1900
@@
 	1    0    0    -1
 $EndComp
-Wire Wire Line
-	10000 6050 10000 6000
-Wire Wire Line
-	10000 6000 9700 6000
 $Comp
 L CONN_01X02 P2
@@
 P 7800 5950
 F 0 "P2" H 7800 6100 50  0000 C CNN
-F 1 "CONN_01X02" V 7900 5950 50  0000 C CNN
+F 1 "BATTERY" V 7900 5950 50  0000 C CNN
 F 2 "SMT_1x2" H 7800 5950 60  0000 C CNN
 F 3 "" H 7800 5950 60  0000 C CNN
@@
 Text GLabel 1100 4150 0    60   Input ~ 0
 VI
-Wire Wire Line
-	8800 6000 8800 6000
 Text GLabel 8800 6000 0    60   Input ~ 0
 EN_B
@@
 Text GLabel 1500 7100 1    60   Input ~ 0
 M0
-Wire Wire Line
-	1500 7100 1500 7150
-Wire Wire Line
-	1400 7150 1600 7150
-Wire Wire Line
-	1600 7150 1600 7200
-Connection ~ 1500 7150
 Text GLabel 1600 7500 3    60   Input ~ 0
 BATT
@@
 Text GLabel 2600 7100 1    60   Input ~ 0
 M1
-Wire Wire Line
-	2600 7100 2600 7150
-Wire Wire Line
-	2500 7150 2700 7150
-Wire Wire Line
-	2700 7150 2700 7200
-Connection ~ 2600 7150
 Text GLabel 2700 7500 3    60   Input ~ 0
 BATT
@@
 Text GLabel 3650 7100 1    60   Input ~ 0
 M2
-Wire Wire Line
-	3650 7100 3650 7150
-Wire Wire Line
-	3550 7150 3750 7150
-Wire Wire Line
-	3750 7150 3750 7200
-Connection ~ 3650 7150
 Text GLabel 3750 7500 3    60   Input ~ 0
 BATT
@@
 Text GLabel 4750 7100 1    60   Input ~ 0
 M3
-Wire Wire Line
-	4750 7100 4750 7150
-Wire Wire Line
-	4650 7150 4850 7150
-Wire Wire Line
-	4850 7150 4850 7200
-Connection ~ 4750 7150
 Text GLabel 4850 7500 3    60   Input ~ 0
 BATT
@@
 	-1   0    0    1
 $EndComp
-Wire Wire Line
-	4100 5100 4100 5200
-Wire Wire Line
-	4100 5150 4050 5150
-Connection ~ 4100 5150
 Text GLabel 4100 4800 1    60   Input ~ 0
 BATT
@@
 Text GLabel 7400 1600 0    60   Input ~ 0
 VI
-Text Notes 2500 4350 0    197  ~ 0
-EXPERIMENTAL\nDO NOT USE\n\nTODO: Add 10u caps + an extra .1u
+Text Notes 11000 4350 0    197  ~ 0
+EXPERIMENTAL\nDO NOT USE\n\nTODO: Add 10u caps + an extra .1u\nTODO: Off-board LEDs
+Text GLabel 5750 2950 2    60   Input ~ 0
+G2
+$Comp
+L LED D7
+U 1 1 57D6EC52
+P 5550 2950
+F 0 "D7" H 5550 3050 50  0000 C CNN
+F 1 "BLU" H 5550 2850 50  0000 C CNN
+F 2 "SM0805" H 5550 2950 60  0000 C CNN
+F 3 "" H 5550 2950 60  0000 C CNN
+	1    5550 2950
+	1    0    0    -1
+$EndComp
+$Comp
+L LED D8
+U 1 1 57D6EF86
+P 5550 3100
+F 0 "D8" H 5550 3200 50  0000 C CNN
+F 1 "BLU" H 5550 3000 50  0000 C CNN
+F 2 "SM0805" H 5550 3100 60  0000 C CNN
+F 3 "" H 5550 3100 60  0000 C CNN
+	1    5550 3100
+	1    0    0    -1
+$EndComp
+$Comp
+L R R7
+U 1 1 57D6F2D5
+P 5200 2950
+F 0 "R7" V 5280 2950 50  0000 C CNN
+F 1 "1.5k" V 5200 2950 50  0000 C CNN
+F 2 "SM0603" V 5130 2950 30  0000 C CNN
+F 3 "" H 5200 2950 30  0000 C CNN
+	1    5200 2950
+	0    -1   -1   0
+$EndComp
+$Comp
+L GND #PWR081
+U 1 1 57D6F41E
+P 5050 3100
+F 0 "#PWR081" H 5050 2850 50  0001 C CNN
+F 1 "GND" H 5050 2950 50  0000 C CNN
+F 2 "" H 5050 3100 60  0000 C CNN
+F 3 "" H 5050 3100 60  0000 C CNN
+	1    5050 3100
+	0    1    1    0
+$EndComp
+Text GLabel 5750 3100 2    60   Input ~ 0
+G2
+$Comp
+L GND #PWR082
+U 1 1 57D6F37D
+P 5050 2950
+F 0 "#PWR082" H 5050 2700 50  0001 C CNN
+F 1 "GND" H 5050 2800 50  0000 C CNN
+F 2 "" H 5050 2950 60  0000 C CNN
+F 3 "" H 5050 2950 60  0000 C CNN
+	1    5050 2950
+	0    1    1    0
+$EndComp
+Wire Wire Line
+	5750 1000 5750 950
+Wire Wire Line
+	5750 950  5600 950
+Wire Wire Line
+	4850 1000 4850 950
+Wire Wire Line
+	4850 950  5000 950
+Wire Wire Line
+	4850 1300 5750 1300
+Wire Wire Line
+	5250 1300 5250 1250
+Connection ~ 5250 1300
+Wire Wire Line
+	5350 1300 5350 1250
+Connection ~ 5350 1300
+Wire Wire Line
+	5600 1300 5600 1350
+Connection ~ 5600 1300
+Wire Wire Line
+	2650 1250 2650 1350
+Wire Wire Line
+	10000 6050 10000 6000
+Wire Wire Line
+	10000 6000 9700 6000
+Wire Wire Line
+	8800 6000 8800 6000
+Wire Wire Line
+	1500 7100 1500 7150
+Wire Wire Line
+	1400 7150 1600 7150
+Wire Wire Line
+	1600 7150 1600 7200
+Connection ~ 1500 7150
+Wire Wire Line
+	2600 7100 2600 7150
+Wire Wire Line
+	2500 7150 2700 7150
+Wire Wire Line
+	2700 7150 2700 7200
+Connection ~ 2600 7150
+Wire Wire Line
+	3650 7100 3650 7150
+Wire Wire Line
+	3550 7150 3750 7150
+Wire Wire Line
+	3750 7150 3750 7200
+Connection ~ 3650 7150
+Wire Wire Line
+	4750 7100 4750 7150
+Wire Wire Line
+	4650 7150 4850 7150
+Wire Wire Line
+	4850 7150 4850 7200
+Connection ~ 4750 7150
+Wire Wire Line
+	4100 5100 4100 5200
+Wire Wire Line
+	4100 5150 4050 5150
+Connection ~ 4100 5150
+$Comp
+L R R6
+U 1 1 57D6F1D8
+P 5200 3100
+F 0 "R6" V 5280 3100 50  0000 C CNN
+F 1 "1.5k" V 5200 3100 50  0000 C CNN
+F 2 "SM0603" V 5130 3100 30  0000 C CNN
+F 3 "" H 5200 3100 30  0000 C CNN
+	1    5200 3100
+	0    -1   -1   0
+$EndComp
+$Comp
+L C E2
+U 1 1 57D7338B
+P 4900 2350
+F 0 "E2" V 4750 2300 50  0000 L CNN
+F 1 "10u" V 4750 2100 50  0000 L CNN
+F 2 "SM0603" H 4938 2200 30  0000 C CNN
+F 3 "" H 4900 2350 60  0000 C CNN
+	1    4900 2350
+	-1   0    0    1
+$EndComp
+$Comp
+L C E1
+U 1 1 57D73642
+P 4650 2350
+F 0 "E1" V 4500 2300 50  0000 L CNN
+F 1 "10u" V 4500 2100 50  0000 L CNN
+F 2 "SM0603" H 4688 2200 30  0000 C CNN
+F 3 "" H 4650 2350 60  0000 C CNN
+	1    4650 2350
+	-1   0    0    1
+$EndComp
+$Comp
+L GND #PWR083
+U 1 1 57D73790
+P 4650 2500
+F 0 "#PWR083" H 4650 2250 50  0001 C CNN
+F 1 "GND" H 4650 2350 50  0000 C CNN
+F 2 "" H 4650 2500 60  0000 C CNN
+F 3 "" H 4650 2500 60  0000 C CNN
+	1    4650 2500
+	1    0    0    -1
+$EndComp
+$Comp
+L GND #PWR084
+U 1 1 57D73837
+P 4900 2500
+F 0 "#PWR084" H 4900 2250 50  0001 C CNN
+F 1 "GND" H 4900 2350 50  0000 C CNN
+F 2 "" H 4900 2500 60  0000 C CNN
+F 3 "" H 4900 2500 60  0000 C CNN
+	1    4900 2500
+	1    0    0    -1
+$EndComp
+$Comp
+L +3.3V #PWR085
+U 1 1 57D73912
+P 4900 2200
+F 0 "#PWR085" H 4900 2050 50  0001 C CNN
+F 1 "+3.3V" H 4900 2340 50  0000 C CNN
+F 2 "" H 4900 2200 60  0000 C CNN
+F 3 "" H 4900 2200 60  0000 C CNN
+	1    4900 2200
+	1    0    0    -1
+$EndComp
+$Comp
+L +3.3V #PWR086
+U 1 1 57D739B9
+P 4650 2200
+F 0 "#PWR086" H 4650 2050 50  0001 C CNN
+F 1 "+3.3V" H 4650 2340 50  0000 C CNN
+F 2 "" H 4650 2200 60  0000 C CNN
+F 3 "" H 4650 2200 60  0000 C CNN
+	1    4650 2200
+	1    0    0    -1
+$EndComp
+$Comp
+L C E3
+U 1 1 57D73A60
+P 5500 2350
+F 0 "E3" V 5350 2300 50  0000 L CNN
+F 1 "100u" V 5350 2100 50  0000 L CNN
+F 2 "C_1206" H 5538 2200 30  0000 C CNN
+F 3 "" H 5500 2350 60  0000 C CNN
+	1    5500 2350
+	-1   0    0    1
+$EndComp
+$Comp
+L GND #PWR087
+U 1 1 57D73CA8
+P 5500 2500
+F 0 "#PWR087" H 5500 2250 50  0001 C CNN
+F 1 "GND" H 5500 2350 50  0000 C CNN
+F 2 "" H 5500 2500 60  0000 C CNN
+F 3 "" H 5500 2500 60  0000 C CNN
+	1    5500 2500
+	1    0    0    -1
+$EndComp
+Text GLabel 5500 2200 1    60   Input ~ 0
+BATT
 $EndSCHEMATC
